File: Splitboard.sch (KiCad schematic (older format))
At the start: 54 parts, among them Y1 16MHz

Commit message: schematic done
Parts:
- added J2: TRRS, symbol Connector:AudioJack4
- added R7, R8: 4.7k, symbol Device:R_Small
- C1, C2, C3, C4, C5, C6, C7: footprint (none) -> Capacitor_SMD:C_0805_2012Metric_Pad1.15x1.40mm_HandSolder
- D0, D1, D10, D11, D12, D2, D20, D21, D22, D30, D31, D32, D40, D41, D42, D50, D51, D52: renamed from D?; footprint (none) -> Diode_SMD:D_0805_2012Metric_Pad1.15x1.40mm_HandSolder
- F1: footprint (none) -> Fuse:Fuse_1206_3216Metric_Pad1.42x1.75mm_HandSolder
- J1: renamed from J?; footprint (none) -> Connector_USB:USB_C_Receptacle_JAE_DX07S016JA1
- KC_A1: renamed from KC_A; footprint (none) -> MX_Only:MXOnly-1U-NoLED
- KC_B1: renamed from KC_B; footprint (none) -> MX_Only:MXOnly-1U-NoLED
- KC_C1: renamed from KC_C; footprint (none) -> MX_Only:MXOnly-1U-NoLED
- KC_D1: renamed from KC_D; footprint (none) -> MX_Only:MXOnly-1U-NoLED
- KC_E1: renamed from KC_E; footprint (none) -> MX_Only:MXOnly-1U-NoLED
- KC_F1: renamed from KC_F; footprint (none) -> MX_Only:MXOnly-1U-NoLED
- KC_G1: renamed from KC_G; footprint (none) -> MX_Only:MXOnly-1U-NoLED
- KC_Q1: renamed from KC_Q; footprint (none) -> MX_Only:MXOnly-1U-NoLED
- KC_R1: renamed from KC_R; footprint (none) -> MX_Only:MXOnly-1U-NoLED
- KC_S1: renamed from KC_S; footprint (none) -> MX_Only:MXOnly-1U-NoLED
- KC_T1: renamed from KC_T; footprint (none) -> MX_Only:MXOnly-1U-NoLED
- KC_V1: renamed from KC_V; footprint (none) -> MX_Only:MXOnly-1U-NoLED
- KC_W1: renamed from KC_W; footprint (none) -> MX_Only:MXOnly-1U-NoLED
- KC_X1: renamed from KC_X; footprint (none) -> MX_Only:MXOnly-1U-NoLED
- KC_Y1: renamed from KC_Y; footprint (none) -> MX_Only:MXOnly-1U-NoLED
- MOD1, MOD2, MOD3: footprint (none) -> MX_Only:MXOnly-1U-NoLED
- R1, R2, R3, R4, R5, R6: footprint (none) -> Resistor_SMD:R_0805_2012Metric_Pad1.15x1.40mm_HandSolder
- SW_RESET1: renamed from SW_RESET; footprint (none) -> Button_Switch_SMD:SW_SPST_TL3342
- Y1: footprint (none) -> Crystal:Crystal_SMD_3225-4Pin_3.2x2.5mm_HandSoldering
- gave numbers to parts that had none: 1
Connections:
- net +5V: now also J2.S, R7.1, R8.1
- net GND: now also J2.T
- net SCL: now reaches U1.18 (PD0)
- net SCL: now also J2.R2, R7.2
- net SDA: now reaches U1.19 (PD1)
- net SDA: now also J2.R1, R8.2
Other:
- moved on the sheet: D0, D1, D10, D11, D12, D2, D20, D21, D22, D30, D31, D32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

Commit message: reupload last save today
Parts:
- R7, R8: footprint (none) -> Resistor_SMD:R_0815_2038Metric_Pad1.53x4.00mm_HandSolder
Changed lines of the file:
@@
 F 0 "R7" H 4409 2296 50  0000 L CNN
 F 1 "4.7k" H 4409 2205 50  0000 L CNN
-F 2 "" H 4350 2250 50  0001 C CNN
+F 2 "Resistor_SMD:R_0815_2038Metric_Pad1.53x4.00mm_HandSolder" H 4350 2250 50  0001 C CNN
 F 3 "~" H 4350 2250 50  0001 C CNN
 	1    4350 2250
@@
 F 0 "R8" H 4109 2296 50  0000 L CNN
 F 1 "4.7k" H 4109 2205 50  0000 L CNN
-F 2 "" H 4050 2250 50  0001 C CNN
+F 2 "Resistor_SMD:R_0815_2038Metric_Pad1.53x4.00mm_HandSolder" H 4050 2250 50  0001 C CNN
 F 3 "~" H 4050 2250 50  0001 C CNN
 	1    4050 2250
@@
 	5550 1800 5700 1800
 $Comp
-L power:GND #PWR?
+L power:GND #PWR0116
 U 1 1 5F621847
 P 5700 2000
-F 0 "#PWR?" H 5700 1750 50  0001 C CNN
+F 0 "#PWR0116" H 5700 1750 50  0001 C CNN
 F 1 "GND" H 5705 1827 50  0000 C CNN
 F 2 "" H 5700 2000 50  0001 C CNN
@@
 	5550 2000 5700 2000
 $Comp
-L power:+5V #PWR?
+L power:+5V #PWR0117
 U 1 1 5F626768
 P 5700 1700
-F 0 "#PWR?" H 5700 1550 50  0001 C CNN
+F 0 "#PWR0117" H 5700 1550 50  0001 C CNN
 F 1 "+5V" H 5715 1873 50  0000 C CNN
 F 2 "" H 5700 1700 50  0001 C CNN
