File: Splitboard_left.sch (KiCad schematic (older format))
At the start: 57 parts, among them J1 USB_C_Receptacle_USB2.0, J2 TRRS, U1 ATmega32U4-AU, Y1 16MHz

Commit message: pcb update
Parts:
- removed J2: TRRS, symbol Connector:AudioJack4
- added D33, D43, D53: SOD-123, Diode_SMD:D_0805_2012Metric_Pad1.15x1.40mm_HandSolder, symbol Device:D_Small
- added J2: TRRS, SJ-43514-SMT:CUI_SJ-43514-SMT, symbol SJ-43514-SMT:SJ-43514-SMT
- added KC_33, KC_43, KC_53: MX-NoLED, MX_Only:MXOnly-1U-NoLED, symbol MX_Alps_Hybrid:MX-NoLED
- R7, R8: footprint Resistor_SMD:R_0815_2038Metric_Pad1.53x4.00mm_HandSolder -> Resistor_SMD:R_0805_2012Metric_Pad1.15x1.40mm_HandSolder
- renumbered KC_Q1 to KC_00, KC_A1 to KC_01, KC_Y1 to KC_02, KC_W1 to KC_10, KC_S1 to KC_11, KC_X1 to KC_12, KC_E1 to KC_20, KC_D1 to KC_21, KC_C1 to KC_22, KC_R1 to KC_30, KC_F1 to KC_31, KC_V1 to KC_32, KC_T1 to KC_40, KC_G1 to KC_41, KC_B1 to KC_42, MOD1 to KC_50, MOD2 to KC_51, MOD3 to KC_52
Connections:
- net +5V: now also J2.1
- net COL3: now also KC_33.1 (COL)
- net COL4: now also KC_43.1 (COL)
- net COL5: now also KC_53.1 (COL)
- net GND: now also J2.2
- net SCL: now also J2.4
- net SDA: now also J2.3
- new net: D53.2 (A), KC_53.2 (ROW)
- new net: D43.2 (A), KC_43.2 (ROW)
- new net: D33.2 (A), KC_33.2 (ROW)
- new net ROW3: D33.1 (K), D43.1 (K), D53.1 (K)
Other:
- moved on the sheet: D0, D1, D10, D11, D12, D2, D20, D21, D22, D30, D31, D32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

Commit message: save
Parts:
- renumbered D0 to D0:0, D1 to D0:1, D2 to D0:2, D10 to D1:0, D11 to D1:1, D12 to D1:2, D20 to D2:0, D21 to D2:1, D22 to D2:2, D30 to D3:0, D31 to D3:1, D32 to D3:2, D33 to D3:3, D40 to D4:0, D41 to D4:1, D42 to D4:2, D43 to D4:3, D50 to D5:0, D51 to D5:1, D52 to D5:2, D53 to D5:3, KC_00 to KC_0:0, KC_01 to KC_0:1, KC_02 to KC_0:2, KC_10 to KC_1:0, KC_11 to KC_1:1, KC_12 to KC_1:2, KC_20 to KC_2:0, KC_21 to KC_2:1, KC_22 to KC_2:2, KC_30 to KC_3:0, KC_31 to KC_3:1, KC_32 to KC_3:2, KC_33 to KC_3:3, KC_40 to KC_4:0, KC_41 to KC_4:1, KC_42 to KC_4:2, KC_43 to KC_4:3, KC_50 to KC_5:0, KC_51 to KC_5:1, KC_52 to KC_5:2, KC_53 to KC_5:3
