File: Splitboard_right.sch (KiCad schematic (older format))
At the start: 69 parts, among them J1 USB_C_Receptacle_USB2.0, J2 TRRS, U1 ATmega32U4-AU, Y1 16MHz

Commit message: save
Parts:
- removed D60, D61, D62: SOD-123, Diode_SMD:D_0805_2012Metric_Pad1.15x1.40mm_HandSolder, symbol Device:D_Small
- removed KC_60, KC_61, KC_62: MX-NoLED, MX_Only:MXOnly-1U-NoLED, symbol MX_Alps_Hybrid:MX-NoLED
- R7, R8: footprint Resistor_SMD:R_0815_2038Metric_Pad1.53x4.00mm_HandSolder -> Resistor_SMD:R_0805_2012Metric_Pad1.15x1.40mm_HandSolder
- renumbered D30 to D10:0, D31 to D10:1, D32 to D10:2, D40 to D11:0, D41 to D11:1, D42 to D11:2, D50 to D12:0, D51 to D12:1, D52 to D12:2, D0 to D7:0, D1 to D7:1, D2 to D7:2, D03 to D7:3, D10 to D8:0, D11 to D8:1, D12 to D8:2, D13 to D8:3, D20 to D9:0, D21 to D9:1, D22 to D9:2, D23 to D9:3, KC_30 to KC_10:0, KC_31 to KC_10:1, KC_32 to KC_10:2, KC_40 to KC_11:0, KC_41 to KC_11:1, KC_42 to KC_11:2, KC_50 to KC_12:0, KC_51 to KC_12:1, KC_52 to KC_12:2, KC_00 to KC_7:0, KC_01 to KC_7:1, KC_02 to KC_7:2, KC_03 to KC_7:3, KC_10 to KC_8:0, KC_11 to KC_8:1, KC_12 to KC_8:2, KC_13 to KC_8:3, KC_20 to KC_9:0, KC_21 to KC_9:1, KC_22 to KC_9:2, KC_23 to KC_9:3
